File: kicad/Router_Lift_Prototype_CNC/Router_Lift_Prototype_CNC.kicad_sch (KiCad schematic)
At the start: 33 parts, among them J1 Conn_01x02, J10 Conn_01x02, J11 Conn_01x04, J2 Conn_01x02, J3 Conn_01x06, J4 Conn_01x06, J5 Conn_01x06, J6 Conn_01x02, J7 Conn_01x02, J8 Conn_01x02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

Commit message: Created the board with DRV8711 Integration
Parts:
- Q1, Q2: footprint Package_TO_SOT_THT:TO-92_Inline -> Package_TO_SOT_THT:TO-92_Inline_Wide
Changed lines of the file:
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@@
       (effects (font (size 1.27 1.27)) (justify left))
     )
-    (property "Footprint" "Package_TO_SOT_THT:TO-92_Inline" (id 2) (at 113.03 179.705 0)
+    (property "Footprint" "Package_TO_SOT_THT:TO-92_Inline_Wide" (id 2) (at 113.03 179.705 0)
       (effects (font (size 1.27 1.27) italic) (justify left) hide)
     )
@@
       (effects (font (size 1.27 1.27)) (justify left))
     )
-    (property "Footprint" "Package_TO_SOT_THT:TO-92_Inline" (id 2) (at 146.05 179.705 0)
+    (property "Footprint" "Package_TO_SOT_THT:TO-92_Inline_Wide" (id 2) (at 146.05 179.705 0)
       (effects (font (size 1.27 1.27) italic) (justify left) hide)
     )
@@
     )
     (path "/964f909b-9a01-49cc-8819-7f4a15220411"
-      (reference "Q1") (unit 1) (value "2N7000") (footprint "Package_TO_SOT_THT:TO-92_Inline")
+      (reference "Q1") (unit 1) (value "2N7000") (footprint "Package_TO_SOT_THT:TO-92_Inline_Wide")
     )
     (path "/fab117e1-2039-4deb-91cb-384068e6600d"
-      (reference "Q2") (unit 1) (value "2N7000") (footprint "Package_TO_SOT_THT:TO-92_Inline")
+      (reference "Q2") (unit 1) (value "2N7000") (footprint "Package_TO_SOT_THT:TO-92_Inline_Wide")
     )
     (path "/f0a78633-40e3-48dc-a667-a550be610cf4"
